File: tcd1304/board/tcd1304_v1.sch (KiCad schematic (older format))
At the start: 25 parts, among them Q1 MMBT3906LT1G, U1 SN74AC14NSR

Commit message: New version for the PCB
Parts:
- CCD1: footprint Package_DIP:DIP-24_W10.16mm -> Package_DIP:DIP-22_W10.16mm_Socket_LongPads
Connections:
- net GNDD: now also U1.1 (1A)
Changed lines of the file:
@@
 F 0 "CCD1" H 9350 3567 50  0000 C CNN
 F 1 "TCD1304" H 9350 3476 50  0000 C CNN
-F 2 "Package_DIP:DIP-24_W10.16mm" H 9300 2850 50  0001 C CNN
+F 2 "Package_DIP:DIP-22_W10.16mm_Socket_LongPads" H 9300 2850 50  0001 C CNN
 F 3 "~" H 9300 2850 50  0001 C CNN
 	1    9300 2850
@@
 $EndComp
 Connection ~ 4400 2350
-Wire Wire Line
-	4400 1650 4400 1700
 Connection ~ 4400 2200
 Connection ~ 4400 1700
@@
 Wire Wire Line
 	9250 1600 9250 2000
+Wire Wire Line
+	4400 1600 4400 1700
 $EndSCHEMATC
